Commit message: Added IMU to urdf description.

File: p3dx_description/urdf/pioneer3dx.urdf (robot description, URDF)
Before this commit: robot pioneer3dx, 11 links, 10 joints
Links:
- added link imu_link
Joints:
- added joint imu_link: type fixed, parent base_link, child imu_link, origin xyz=0 0 0.1 rpy=0 0 0, axis 0 0 0
